File: Keyboard_60%.kicad_pcb (KiCad board)
At the start: 2 copper layers, 284.7 x 94.2 mm, 0 parts

Commit message: Placed switches
Parts:
- added AE1: Antenna_Shield, keyboard:BLE_ANTENNA, F.Cu at (432.7, 310.6)
- added C1: 1uF, keyboard:C_0603_1608Metric, F.Cu at (476.6, 308.2)
- added C10: 0.8pF, keyboard:C_0402_1005Metric, F.Cu at (450.0, 305.4)
- added C11: 0.5pF, keyboard:C_0402_1005Metric, F.Cu at (450.0, 307.3)
- added C12: DNP, keyboard:C_0402_1005Metric, F.Cu at (450.0, 309.3)
- added C13: 100pF, keyboard:C_0402_1005Metric, F.Cu at (450.0, 311.3)
- added C14: 1uF, keyboard:C_0603_1608Metric, F.Cu at (455.7, 298.2)
- added C15: DNP, keyboard:C_0402_1005Metric, F.Cu at (450.0, 313.2)
- added C16: 100nF, keyboard:C_0402_1005Metric, F.Cu at (470.2, 318.0)
- added C2: 4u7F, keyboard:C_0805_2012Metric, F.Cu at (480.8, 318.1)
- added C20: 4u7F, keyboard:C_0805_2012Metric, F.Cu at (447.9, 315.7)
- added C21: 4u7F, keyboard:C_0805_2012Metric, F.Cu at (447.9, 318.7)
- added C22: 4u7F, keyboard:C_0805_2012Metric, F.Cu at (447.9, 321.7)
- added C23: 1uF, keyboard:C_0603_1608Metric, F.Cu at (455.7, 300.7)
- added C24: 100nF, keyboard:C_0402_1005Metric, F.Cu at (452.9, 305.4)
- added C25: 100nF, keyboard:C_0402_1005Metric, F.Cu at (452.9, 307.3)
- added C26: 100nF, keyboard:C_0402_1005Metric, F.Cu at (452.9, 309.3)
- added C27: 100nF, keyboard:C_0402_1005Metric, F.Cu at (452.9, 311.3)
- added C3: 1uF, keyboard:C_0603_1608Metric, F.Cu at (476.6, 310.7)
- added C4: 1uF, keyboard:C_0603_1608Metric, F.Cu at (476.6, 313.2)
- added C5: 100nF, keyboard:C_0402_1005Metric, F.Cu at (447.2, 305.4)
- added C6: 100nF, keyboard:C_0402_1005Metric, F.Cu at (447.2, 307.3)
- added C7: 100nF, keyboard:C_0402_1005Metric, F.Cu at (447.2, 309.3)
- added C8: 100nF, keyboard:C_0402_1005Metric, F.Cu at (447.2, 311.3)
- added C9: 820pF, keyboard:C_0402_1005Metric, F.Cu at (447.2, 313.2)
- added D1: LED, keyboard:LED_0603_1608Metric, F.Cu at (480.6, 312.7)
- added D10: 1N4148, Diode_THT:D_DO-35_SOD27_P7.62mm_Horizontal, F.Cu at (631.9, 139.7)
- added D11: 1N4148, Diode_THT:D_DO-35_SOD27_P7.62mm_Horizontal, F.Cu at (631.9, 143.3)
- added D12: 1N4148, Diode_THT:D_DO-35_SOD27_P7.62mm_Horizontal, F.Cu at (631.9, 146.8)
- added D13: 1N4148, Diode_THT:D_DO-35_SOD27_P7.62mm_Horizontal, F.Cu at (631.9, 150.4)
- added D14: 1N4148, Diode_THT:D_DO-35_SOD27_P7.62mm_Horizontal, F.Cu at (631.9, 153.9)
- added D15: 1N4148, Diode_THT:D_DO-35_SOD27_P7.62mm_Horizontal, F.Cu at (631.9, 157.5)
- added D16: 1N4148, Diode_THT:D_DO-35_SOD27_P7.62mm_Horizontal, F.Cu at (642.7, 114.9)
- added D17: 1N4148, Diode_THT:D_DO-35_SOD27_P7.62mm_Horizontal, F.Cu at (642.7, 118.4)
- added D18: 1N4148, Diode_THT:D_DO-35_SOD27_P7.62mm_Horizontal, F.Cu at (642.7, 122.0)
- added D19: 1N4148, Diode_THT:D_DO-35_SOD27_P7.62mm_Horizontal, F.Cu at (642.7, 125.5)
- added D2: LED, keyboard:LED_0603_1608Metric, F.Cu at (480.6, 315.3)
- added D20: 1N4148, Diode_THT:D_DO-35_SOD27_P7.62mm_Horizontal, F.Cu at (642.7, 129.1)
- added D21: 1N4148, Diode_THT:D_DO-35_SOD27_P7.62mm_Horizontal, F.Cu at (642.7, 132.6)
- added D22: 1N4148, Diode_THT:D_DO-35_SOD27_P7.62mm_Horizontal, F.Cu at (642.7, 136.2)
- added D23: 1N4148, Diode_THT:D_DO-35_SOD27_P7.62mm_Horizontal, F.Cu at (642.7, 139.7)
- added D24: 1N4148, Diode_THT:D_DO-35_SOD27_P7.62mm_Horizontal, F.Cu at (642.7, 143.3)
- added D25: 1N4148, Diode_THT:D_DO-35_SOD27_P7.62mm_Horizontal, F.Cu at (642.7, 146.8)
- added D26: 1N4148, Diode_THT:D_DO-35_SOD27_P7.62mm_Horizontal, F.Cu at (642.7, 150.4)
- added D27: 1N4148, Diode_THT:D_DO-35_SOD27_P7.62mm_Horizontal, F.Cu at (642.7, 153.9)
- added D28: 1N4148, Diode_THT:D_DO-35_SOD27_P7.62mm_Horizontal, F.Cu at (642.7, 157.5)
- added D29: 1N4148, Diode_THT:D_DO-35_SOD27_P7.62mm_Horizontal, F.Cu at (653.5, 114.9)
- added D3: 1N4148, Diode_THT:D_DO-35_SOD27_P7.62mm_Horizontal, F.Cu at (631.9, 114.9)
- added D30: 1N4148, Diode_THT:D_DO-35_SOD27_P7.62mm_Horizontal, F.Cu at (653.5, 118.4)
- added D31: 1N4148, Diode_THT:D_DO-35_SOD27_P7.62mm_Horizontal, F.Cu at (653.5, 122.0)
- added D32: 1N4148, Diode_THT:D_DO-35_SOD27_P7.62mm_Horizontal, F.Cu at (653.5, 125.5)
- added D33: 1N4148, Diode_THT:D_DO-35_SOD27_P7.62mm_Horizontal, F.Cu at (653.5, 129.1)
- added D34: 1N4148, Diode_THT:D_DO-35_SOD27_P7.62mm_Horizontal, F.Cu at (653.5, 132.6)
- added D35: 1N4148, Diode_THT:D_DO-35_SOD27_P7.62mm_Horizontal, F.Cu at (653.5, 136.2)
- added D36: 1N4148, Diode_THT:D_DO-35_SOD27_P7.62mm_Horizontal, F.Cu at (653.5, 139.7)
- added D37: 1N4148, Diode_THT:D_DO-35_SOD27_P7.62mm_Horizontal, F.Cu at (653.5, 143.3)
- added D38: 1N4148, Diode_THT:D_DO-35_SOD27_P7.62mm_Horizontal, F.Cu at (653.5, 146.8)
- added D39: 1N4148, Diode_THT:D_DO-35_SOD27_P7.62mm_Horizontal, F.Cu at (653.5, 150.4)
- added D4: 1N4148, Diode_THT:D_DO-35_SOD27_P7.62mm_Horizontal, F.Cu at (631.9, 118.4)
- added D40: 1N4148, Diode_THT:D_DO-35_SOD27_P7.62mm_Horizontal, F.Cu at (653.5, 153.9)
- added D41: 1N4148, Diode_THT:D_DO-35_SOD27_P7.62mm_Horizontal, F.Cu at (653.5, 157.5)
- added D42: 1N4148, Diode_THT:D_DO-35_SOD27_P7.62mm_Horizontal, F.Cu at (664.2, 114.9)
- added D43: 1N4148, Diode_THT:D_DO-35_SOD27_P7.62mm_Horizontal, F.Cu at (664.2, 118.4)
- added D44: 1N4148, Diode_THT:D_DO-35_SOD27_P7.62mm_Horizontal, F.Cu at (664.2, 122.0)
- added D45: 1N4148, Diode_THT:D_DO-35_SOD27_P7.62mm_Horizontal, F.Cu at (664.2, 125.5)
- added D46: 1N4148, Diode_THT:D_DO-35_SOD27_P7.62mm_Horizontal, F.Cu at (664.2, 129.1)
- added D47: 1N4148, Diode_THT:D_DO-35_SOD27_P7.62mm_Horizontal, F.Cu at (664.2, 132.6)
- added D48: 1N4148, Diode_THT:D_DO-35_SOD27_P7.62mm_Horizontal, F.Cu at (664.2, 136.2)
- added D49: 1N4148, Diode_THT:D_DO-35_SOD27_P7.62mm_Horizontal, F.Cu at (664.2, 139.7)
- added D5: 1N4148, Diode_THT:D_DO-35_SOD27_P7.62mm_Horizontal, F.Cu at (631.9, 122.0)
- added D50: 1N4148, Diode_THT:D_DO-35_SOD27_P7.62mm_Horizontal, F.Cu at (664.2, 143.3)
- added D51: 1N4148, Diode_THT:D_DO-35_SOD27_P7.62mm_Horizontal, F.Cu at (664.2, 146.8)
- added D52: 1N4148, Diode_THT:D_DO-35_SOD27_P7.62mm_Horizontal, F.Cu at (664.2, 150.4)
- added D53: 1N4148, Diode_THT:D_DO-35_SOD27_P7.62mm_Horizontal, F.Cu at (664.2, 153.9)
- added D54: 1N4148, Diode_THT:D_DO-35_SOD27_P7.62mm_Horizontal, F.Cu at (664.2, 157.5)
- added D55: 1N4148, Diode_THT:D_DO-35_SOD27_P7.62mm_Horizontal, F.Cu at (675.0, 114.9)
- added D56: 1N4148, Diode_THT:D_DO-35_SOD27_P7.62mm_Horizontal, F.Cu at (675.0, 118.4)
- added D57: 1N4148, Diode_THT:D_DO-35_SOD27_P7.62mm_Horizontal, F.Cu at (675.0, 122.0)
- added D58: 1N4148, Diode_THT:D_DO-35_SOD27_P7.62mm_Horizontal, F.Cu at (675.0, 125.5)
- added D59: 1N4148, Diode_THT:D_DO-35_SOD27_P7.62mm_Horizontal, F.Cu at (675.0, 129.1)
- added D6: 1N4148, Diode_THT:D_DO-35_SOD27_P7.62mm_Horizontal, F.Cu at (631.9, 125.5)
- added D60: 1N4148, Diode_THT:D_DO-35_SOD27_P7.62mm_Horizontal, F.Cu at (675.0, 132.6)
- added D61: 1N4148, Diode_THT:D_DO-35_SOD27_P7.62mm_Horizontal, F.Cu at (675.0, 136.2)
- added D62: 1N4148, Diode_THT:D_DO-35_SOD27_P7.62mm_Horizontal, F.Cu at (675.0, 139.7)
- added D63: 1N4148, Diode_THT:D_DO-35_SOD27_P7.62mm_Horizontal, F.Cu at (675.0, 143.3)
- added D64: 1N4148, Diode_THT:D_DO-35_SOD27_P7.62mm_Horizontal, F.Cu at (675.0, 146.8)
- added D65: 1N4148, Diode_THT:D_DO-35_SOD27_P7.62mm_Horizontal, F.Cu at (675.0, 150.4)
- added D7: 1N4148, Diode_THT:D_DO-35_SOD27_P7.62mm_Horizontal, F.Cu at (631.9, 129.1)
- added D8: 1N4148, Diode_THT:D_DO-35_SOD27_P7.62mm_Horizontal, F.Cu at (631.9, 132.6)
- added D9: 1N4148, Diode_THT:D_DO-35_SOD27_P7.62mm_Horizontal, F.Cu at (631.9, 136.2)
- added J1: JST-4-pin, keyboard:JST-4-pin, F.Cu at (464.6, 308.5)
- added J2: JST-2-pin, keyboard:JST-2-pin, F.Cu at (471.6, 310.2)
- added J3: Prog_conn, keyboard:DB_CONN, F.Cu at (439.6, 300.6)
- added J4: TYPE-C-31-M12_13, keyboard:tyye_c_connector, F.Cu at (466.5, 303.6)
- added J5: Tag connect TC2030-CTX, keyboard:TC2030-IDC-NL, F.Cu at (454.3, 316.8)
- added JP1: SolderJumper, keyboard:SolderBridge, F.Cu at (452.3, 321.2)
- added L1: 4.7nH, keyboard:L_0402_1005Metric, F.Cu at (441.1, 312.4)
- added L2: 60R@100MHz, Inductor_SMD:L_1206_3216Metric, F.Cu at (471.6, 315.2)
- added MX1: 1u, keyboard:SW_Cherry_MX_1.00u_PCB, F.Cu at (90.2, 90.7)
- added MX10: 1u, keyboard:SW_Cherry_MX_1.00u_PCB, F.Cu at (261.3, 90.7)
- added MX11: 1u, keyboard:SW_Cherry_MX_1.00u_PCB, F.Cu at (280.4, 90.7)
- added MX12: 1u, keyboard:SW_Cherry_MX_1.00u_PCB, F.Cu at (299.5, 90.7)
- added MX13: 1u, keyboard:SW_Cherry_MX_1.00u_PCB, F.Cu at (318.7, 90.7)
- added MX14: 1u, keyboard:SW_Cherry_MX_1.00u_PCB, F.Cu at (337.8, 90.7)
- added MX15: 1u, keyboard:SW_Cherry_MX_1.00u_PCB, F.Cu at (356.9, 90.7)
- added MX16: 2u, keyboard:SW_Cherry_MX_2.00u_PCB, F.Cu at (347.3, 90.8)
- added MX17: 1.5u, keyboard:SW_Cherry_MX_1.50u_PCB, F.Cu at (95.0, 109.8)
- added MX18: 1u, keyboard:SW_Cherry_MX_1.00u_PCB, F.Cu at (118.8, 109.8)
- added MX19: 1u, keyboard:SW_Cherry_MX_1.00u_PCB, F.Cu at (137.7, 109.8)
- added MX2: 1u, keyboard:SW_Cherry_MX_1.00u_PCB, F.Cu at (109.2, 90.7)
- added MX20: 1u, keyboard:SW_Cherry_MX_1.00u_PCB, F.Cu at (156.7, 109.8)
- added MX21: 1u, keyboard:SW_Cherry_MX_1.00u_PCB, F.Cu at (175.7, 109.8)
- added MX22: 1u, keyboard:SW_Cherry_MX_1.00u_PCB, F.Cu at (194.7, 109.8)
- added MX23: 1u, keyboard:SW_Cherry_MX_1.00u_PCB, F.Cu at (213.7, 109.8)
- added MX24: 1u, keyboard:SW_Cherry_MX_1.00u_PCB, F.Cu at (232.7, 109.8)
- added MX25: 1u, keyboard:SW_Cherry_MX_1.00u_PCB, F.Cu at (251.7, 109.8)
- added MX26: 1u, keyboard:SW_Cherry_MX_1.00u_PCB, F.Cu at (270.7, 109.8)
- added MX27: 1u, keyboard:SW_Cherry_MX_1.00u_PCB, F.Cu at (289.7, 109.8)
- added MX28: 1u, keyboard:SW_Cherry_MX_1.00u_PCB, F.Cu at (308.9, 109.8)
- added MX29: 1u, keyboard:SW_Cherry_MX_1.00u_PCB, F.Cu at (328.2, 109.8)
- added MX3: 1u, keyboard:SW_Cherry_MX_1.00u_PCB, F.Cu at (128.2, 90.7)
- added MX30: 1.5u, keyboard:SW_Cherry_MX_1.50u_PCB, F.Cu at (352.1, 109.8)
- added MX31: 1.75u, keyboard:SW_Cherry_MX_1.75u_PCB, F.Cu at (97.4, 128.8)
- added MX32: 1.25u, keyboard:SW_Cherry_MX_1.25u_PCB, F.Cu at (92.6, 128.8)
- added MX33: 1u, keyboard:SW_Cherry_MX_1.00u_PCB, F.Cu at (123.6, 128.8)
- added MX34: 1u, keyboard:SW_Cherry_MX_1.00u_PCB, F.Cu at (142.7, 128.8)
- added MX35: 1u, keyboard:SW_Cherry_MX_1.00u_PCB, F.Cu at (161.8, 128.8)
- added MX36: 1u, keyboard:SW_Cherry_MX_1.00u_PCB, F.Cu at (180.9, 128.8)
- added MX37: 1u, keyboard:SW_Cherry_MX_1.00u_PCB, F.Cu at (199.9, 128.8)
- added MX38: 1u, keyboard:SW_Cherry_MX_1.00u_PCB, F.Cu at (218.9, 128.8)
- added MX39: 1u, keyboard:SW_Cherry_MX_1.00u_PCB, F.Cu at (238.0, 128.8)
- added MX4: 1u, keyboard:SW_Cherry_MX_1.00u_PCB, F.Cu at (147.2, 90.7)
- added MX40: 1u, keyboard:SW_Cherry_MX_1.00u_PCB, F.Cu at (257.0, 128.8)
- added MX41: 1u, keyboard:SW_Cherry_MX_1.00u_PCB, F.Cu at (276.0, 128.8)
- added MX42: 1u, keyboard:SW_Cherry_MX_1.00u_PCB, F.Cu at (295.0, 128.8)
- added MX43: 1u, keyboard:SW_Cherry_MX_1.00u_PCB, F.Cu at (314.0, 128.8)
- added MX44: 2.25u, keyboard:SW_Cherry_MX_2.25u_PCB, F.Cu at (345.0, 128.8)
- added MX45: 2.25u, keyboard:SW_Cherry_MX_2.25u_PCB, F.Cu at (102.1, 147.8)
- added MX46: 1u, keyboard:SW_Cherry_MX_1.00u_PCB, F.Cu at (133.1, 147.8)
- added MX47: 1u, keyboard:SW_Cherry_MX_1.00u_PCB, F.Cu at (152.2, 147.8)
- added MX48: 1u, keyboard:SW_Cherry_MX_1.00u_PCB, F.Cu at (171.2, 147.8)
- added MX49: 1u, keyboard:SW_Cherry_MX_1.00u_PCB, F.Cu at (190.3, 147.8)
- added MX5: 1u, keyboard:SW_Cherry_MX_1.00u_PCB, F.Cu at (166.2, 90.7)
- added MX50: 1u, keyboard:SW_Cherry_MX_1.00u_PCB, F.Cu at (209.4, 147.8)
- added MX51: 1u, keyboard:SW_Cherry_MX_1.00u_PCB, F.Cu at (228.5, 147.8)
- added MX52: 1u, keyboard:SW_Cherry_MX_1.00u_PCB, F.Cu at (247.6, 147.8)
- added MX53: 1u, keyboard:SW_Cherry_MX_1.00u_PCB, F.Cu at (266.6, 147.8)
- added MX54: 1u, keyboard:SW_Cherry_MX_1.00u_PCB, F.Cu at (285.7, 147.8)
- added MX55: 1u, keyboard:SW_Cherry_MX_1.00u_PCB, F.Cu at (304.7, 147.8)
- added MX56: 1.75u, keyboard:SW_Cherry_MX_1.75u_PCB, F.Cu at (330.8, 147.8)
- added MX57: 1u, keyboard:SW_Cherry_MX_1.00u_PCB, F.Cu at (356.9, 147.8)
- added MX58: 2.75u, keyboard:SW_Cherry_MX_2.75u_PCB, F.Cu at (340.2, 147.8)
- added MX59: 1.25u, keyboard:SW_Cherry_MX_1.25u_PCB, F.Cu at (92.6, 166.8)
- added MX6: 1u, keyboard:SW_Cherry_MX_1.00u_PCB, F.Cu at (185.2, 90.7)
- added MX60: 1.25u, keyboard:SW_Cherry_MX_1.25u_PCB, F.Cu at (116.4, 166.8)
- added MX61: 1.25u, keyboard:SW_Cherry_MX_1.25u_PCB, F.Cu at (140.2, 166.8)
- added MX62: 1.5u, keyboard:SW_Cherry_MX_1.50u_PCB, F.Cu at (95.0, 166.9)
- added MX63: 1.5u, keyboard:SW_Cherry_MX_1.50u_PCB, F.Cu at (123.5, 166.9)
- added MX64: 1.5u, keyboard:SW_Cherry_MX_1.50u_PCB, F.Cu at (152.0, 166.9)
- added MX65: 6.25u, keyboard:SW_Cherry_MX_6.25u_PCB, F.Cu at (211.7, 166.8)
- added MX66: 7u, keyboard:SW_Cherry_MX_7.00u_PCB, F.Cu at (230.5, 171.9)
- added MX67: 1.25u, keyboard:SW_Cherry_MX_1.25u_PCB, F.Cu at (283.1, 166.8)
- added MX68: 1.25u, keyboard:SW_Cherry_MX_1.25u_PCB, F.Cu at (306.9, 166.8)
- added MX69: 1.25u, keyboard:SW_Cherry_MX_1.25u_PCB, F.Cu at (330.8, 166.8)
- added MX7: 1u, keyboard:SW_Cherry_MX_1.00u_PCB, F.Cu at (204.2, 90.7)
- added MX70: 1.25u, keyboard:SW_Cherry_MX_1.25u_PCB, F.Cu at (354.5, 166.8)
- added MX71: 1.5u, keyboard:SW_Cherry_MX_1.50u_PCB, F.Cu at (314.0, 166.8)
- added MX72: 1u, keyboard:SW_Cherry_MX_1.00u_PCB, F.Cu at (337.8, 166.9)
- added MX73: 1u, keyboard:SW_Cherry_MX_1.00u_PCB, F.Cu at (356.9, 166.9)
- added MX8: 1u, keyboard:SW_Cherry_MX_1.00u_PCB, F.Cu at (223.2, 90.7)
- added MX9: 1u, keyboard:SW_Cherry_MX_1.00u_PCB, F.Cu at (242.2, 90.7)
- added R1: 1k2, keyboard:R_0402_1005Metric, F.Cu at (477.5, 297.9)
- added R10: 22E, keyboard:R_0402_1005Metric, F.Cu at (444.1, 312.4)
- added R11: 22E, keyboard:R_0402_1005Metric, F.Cu at (444.1, 314.4)
- added R12: 22E, keyboard:R_0402_1005Metric, F.Cu at (444.1, 316.3)
- added R13: 10k, keyboard:R_0402_1005Metric, F.Cu at (444.1, 318.3)
- added R14: 10k, keyboard:R_0402_1005Metric, F.Cu at (480.4, 297.9)
- added R15: 10k, keyboard:R_0402_1005Metric, F.Cu at (480.4, 299.9)
- added R16: 5k1, keyboard:R_0402_1005Metric, F.Cu at (480.4, 301.9)
- added R17: 5k1, keyboard:R_0402_1005Metric, F.Cu at (480.4, 303.9)
- added R18: 10k, keyboard:R_0402_1005Metric, F.Cu at (444.1, 320.3)
- added R2: 1k2, keyboard:R_0402_1005Metric, F.Cu at (477.5, 299.9)
- added R3: 1k2, keyboard:R_0402_1005Metric, F.Cu at (477.5, 301.9)
- added R4: 1k2, keyboard:R_0402_1005Metric, F.Cu at (477.5, 303.9)
- added R5: 5k1, keyboard:R_0402_1005Metric, F.Cu at (477.5, 305.9)
- added R6: 22E, keyboard:R_0402_1005Metric, F.Cu at (441.1, 314.4)
- added R7: 22E, keyboard:R_0402_1005Metric, F.Cu at (441.1, 316.3)
- added R8: 10k, keyboard:R_0402_1005Metric, F.Cu at (441.1, 318.3)
- added R9: 10k, keyboard:R_0402_1005Metric, F.Cu at (441.1, 320.3)
- added TH1: 10k, keyboard:R_0402_1005Metric, F.Cu at (480.4, 305.9)
- added U1: BQ24074RGTR, keyboard:QFN-16, F.Cu at (463.6, 316.7)
- added U2: AP2127K-3.0TRG1, keyboard:SOT-23-5, F.Cu at (481.1, 309.2)
- added U3: NRF52840-QIAA-R, keyboard:aqfn73, F.Cu at (434.7, 316.4)
- added U4: TPD4E05U06DQAR, keyboard:USON-10, F.Cu at (476.6, 316.5)
- added Y1: 32MHz, keyboard:SMD-4_crystal, F.Cu at (451.3, 299.0)
- added Y2: 32.768kHz, keyboard:SMD-2_crystal, F.Cu at (450.6, 302.4)

Commit message: Pcb routing complete
Parts:
- removed J1: JST-4-pin, keyboard:JST-4-pin
- removed J2: JST-2-pin, keyboard:JST-2-pin
- added BT1: Lipo cell, keyboard:JST-2-pin, B.Cu at (137.0, 125.0)
- added R19: 10k, keyboard:R_0402_1005Metric, B.Cu at (92.8, 102.6)
- added R20: 10k, keyboard:R_0402_1005Metric, B.Cu at (98.1, 107.6)
- added R21: 10k, keyboard:R_0402_1005Metric, B.Cu at (92.2, 136.8)
- added R22: 10k, keyboard:R_0402_1005Metric, B.Cu at (91.3, 155.2)
- added R23: 10k, keyboard:R_0402_1005Metric, B.Cu at (81.8, 167.8)
- AE1, C1, C10, C11, C12, C13, C14, C15, C16, C2, C20, C21, C22, C23, C24, C25, C26, C27, C3, C4, C5, C6, C7, C8, C9, J4, JP1, L1, R1, R10, R11, R12, R13, R14, R15, R16, R17, R18, R2, R3, R4, R5, R6, R7, R8, R9, TH1, U1, U2, U3, U4, Y1, Y2: moved to B.Cu
- D10, D11, D12, D13, D14, D15, D16, D17, D18, D19, D20, D21, D22, D23, D24, D25, D26, D27, D28, D29, D3, D30, D31, D32, D33, D34, D35, D36, D37, D38, D39, D4, D40, D41, D42, D43, D44, D45, D46, D47, D48, D49, D5, D50, D51, D52, D53, D54, D55, D56, D57, D58, D59, D6, D60, D61, D62, D63, D64, D65, D7, D8, D9: footprint Diode_THT:D_DO-35_SOD27_P7.62mm_Horizontal -> keyboard:D_SOD-123; moved to B.Cu
- L2: footprint Inductor_SMD:L_1206_3216Metric -> keyboard:L_0603_1608Metric; moved to B.Cu
- MX62: value 1.5u -> 6.25u; footprint keyboard:SW_Cherry_MX_1.50u_PCB -> keyboard:SW_Cherry_MX_6.25u_PCB
- MX63, MX64: value 1.5u -> 1.25u; footprint keyboard:SW_Cherry_MX_1.50u_PCB -> keyboard:SW_Cherry_MX_1.25u_PCB
- MX65: value 6.25u -> 1.25u; footprint keyboard:SW_Cherry_MX_6.25u_PCB -> keyboard:SW_Cherry_MX_1.25u_PCB
- MX66: value 7u -> 1.25u; footprint keyboard:SW_Cherry_MX_7.00u_PCB -> keyboard:SW_Cherry_MX_1.25u_PCB
- MX67, MX68, MX69: value 1.25u -> 1.5u; footprint keyboard:SW_Cherry_MX_1.25u_PCB -> keyboard:SW_Cherry_MX_1.50u_PCB
- MX70: value 1.25u -> 7u; footprint keyboard:SW_Cherry_MX_1.25u_PCB -> keyboard:SW_Cherry_MX_7.00u_PCB
- moved D58 595.5 mm to (81.2, 171.0), turned to 90 degrees
- moved D45 573.0 mm to (91.8, 152.0), turned to 90 degrees
- moved D59 572.2 mm to (104.3, 170.9), turned to 90 degrees
- moved D32 565.3 mm to (88.3, 138.4), turned to 180 degrees
- moved D18 554.2 mm to (88.7, 107.9), turned to -90 degrees
- moved D60 547.4 mm to (129.0, 171.0), turned to 90 degrees
- moved D3 545.9 mm to (86.2, 100.8), turned to 180 degrees
- moved D46 542.2 mm to (122.5, 151.9), turned to 90 degrees
- moved D33 540.1 mm to (113.4, 134.7), turned to 90 degrees
- moved D19 530.6 mm to (112.4, 107.9), turned to -90 degrees
- moved D47 523.2 mm to (141.4, 152.0), turned to 90 degrees
- moved D34 521.5 mm to (131.9, 132.9), turned to 90 degrees
- moved D4 517.9 mm to (114.5, 95.5), turned to 90 degrees
- moved D5 515.2 mm to (117.4, 95.5), turned to 90 degrees
- moved D20 511.7 mm to (131.4, 107.9), turned to -90 degrees
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Connections:
- net Net-(AE1-A) renamed /ANT_FEED
- D10 pad 1: /ROW0 -> /switch_matrix/ROW0
- D11 pad 1: /ROW0 -> /switch_matrix/ROW0
- D12 pad 1: /ROW0 -> /switch_matrix/ROW0
- D13 pad 1: /ROW0 -> /switch_matrix/ROW0
- D14 pad 1: /ROW0 -> /switch_matrix/ROW0
- D15 pad 1: /ROW0 -> /switch_matrix/ROW0
- D16 pad 1: /ROW0 -> /switch_matrix/ROW0
- D17 pad 1: /ROW0 -> /switch_matrix/ROW0
- D18 pad 1: /ROW1 -> /switch_matrix/ROW1
- D19 pad 1: /ROW1 -> /switch_matrix/ROW1
- D20 pad 1: /ROW1 -> /switch_matrix/ROW1
- D21 pad 1: /ROW1 -> /switch_matrix/ROW1
- D22 pad 1: /ROW1 -> /switch_matrix/ROW1
- D23 pad 1: /ROW1 -> /switch_matrix/ROW1
- D24 pad 1: /ROW1 -> /switch_matrix/ROW1
- D25 pad 1: /ROW1 -> /switch_matrix/ROW1
- D26 pad 1: /ROW1 -> /switch_matrix/ROW1
- D27 pad 1: /ROW1 -> /switch_matrix/ROW1
- D28 pad 1: /ROW1 -> /switch_matrix/ROW1
- D29 pad 1: /ROW1 -> /switch_matrix/ROW1
- D3 pad 1: /ROW0 -> /switch_matrix/ROW0
- D30 pad 1: /ROW1 -> /switch_matrix/ROW1
- D31 pad 1: /ROW1 -> /switch_matrix/ROW1
- D32 pad 1: /ROW2 -> /switch_matrix/ROW2
- D33 pad 1: /ROW2 -> /switch_matrix/ROW2
- D34 pad 1: /ROW2 -> /switch_matrix/ROW2
- D35 pad 1: unconnected-(D35-K-Pad1) -> /switch_matrix/ROW2
- D36 pad 1: /ROW2 -> /switch_matrix/ROW2
- D37 pad 1: /ROW2 -> /switch_matrix/ROW2
- D38 pad 1: /ROW2 -> /switch_matrix/ROW2
- D39 pad 1: /ROW2 -> /switch_matrix/ROW2
- D4 pad 1: /ROW0 -> /switch_matrix/ROW0
- D40 pad 1: /ROW2 -> /switch_matrix/ROW2
- D41 pad 1: /ROW2 -> /switch_matrix/ROW2
- D42 pad 1: /ROW2 -> /switch_matrix/ROW2
- D43 pad 1: /ROW2 -> /switch_matrix/ROW2
- D44 pad 1: /ROW2 -> /switch_matrix/ROW2
- D45 pad 1: /ROW3 -> /switch_matrix/ROW3
- D46 pad 1: /ROW3 -> /switch_matrix/ROW3
- D47 pad 1: /ROW3 -> /switch_matrix/ROW3
- D48 pad 1: /ROW3 -> /switch_matrix/ROW3
- D49 pad 1: /ROW3 -> /switch_matrix/ROW3
- D5 pad 1: /ROW0 -> /switch_matrix/ROW0
- D50 pad 1: /ROW3 -> /switch_matrix/ROW3
- D51 pad 1: /ROW3 -> /switch_matrix/ROW3
- D52 pad 1: /ROW3 -> /switch_matrix/ROW3
- D53 pad 1: /ROW3 -> /switch_matrix/ROW3
- D54 pad 1: /ROW3 -> /switch_matrix/ROW3
- D55 pad 1: /ROW3 -> /switch_matrix/ROW3
- D56 pad 1: /ROW3 -> /switch_matrix/ROW3
- D57 pad 1: /ROW3 -> /switch_matrix/ROW3
- D58 pad 1: /ROW4 -> /switch_matrix/ROW4
- D59 pad 1: /ROW4 -> /switch_matrix/ROW4
- D6 pad 1: /ROW0 -> /switch_matrix/ROW0
- D60 pad 1: /ROW4 -> /switch_matrix/ROW4
- D61 pad 1: /ROW4 -> /switch_matrix/ROW4
- D62 pad 1: /ROW4 -> /switch_matrix/ROW4
- D63 pad 1: /ROW4 -> /switch_matrix/ROW4
- D64 pad 1: /ROW4 -> /switch_matrix/ROW4
- D65 pad 1: /ROW4 -> /switch_matrix/ROW4
- D7 pad 1: /ROW0 -> /switch_matrix/ROW0
- D8 pad 1: /ROW0 -> /switch_matrix/ROW0
- D9 pad 1: /ROW0 -> /switch_matrix/ROW0
- J5 pad 1: /3V3 -> Net-(J5-Pin_1)
- J5 pad 3: /nReset -> /~{nReset}
- JP1 pad 2: Net-(JP1-B) -> Net-(J5-Pin_1)
- MX13 pad 1: /COL12 -> Net-(D15-A)
- MX13 pad 2: Net-(D15-A) -> /COL12
- MX62 pad 1: Net-(D58-A) -> Net-(D61-A)
- MX62 pad 2: /COL0 -> /COL6
- MX63 pad 1: Net-(D59-A) -> Net-(D62-A)
- MX63 pad 2: /COL1 -> /COL10
- MX64 pad 1: Net-(D60-A) -> Net-(D63-A)
- MX64 pad 2: /COL2 -> /COL11
- MX65 pad 1: Net-(D61-A) -> Net-(D64-A)
- MX65 pad 2: /COL6 -> /COL12
- MX66 pad 1: Net-(D61-A) -> Net-(D65-A)
- MX66 pad 2: /COL6 -> /COL13
- MX67 pad 1: Net-(D62-A) -> Net-(D58-A)
- MX67 pad 2: /COL10 -> /COL0
- MX68 pad 1: Net-(D63-A) -> Net-(D59-A)
- MX68 pad 2: /COL11 -> /COL1
- MX69 pad 1: Net-(D64-A) -> Net-(D60-A)
- MX69 pad 2: /COL12 -> /COL2
- MX70 pad 1: Net-(D65-A) -> Net-(D61-A)
- MX70 pad 2: /COL13 -> /COL6
- R13 pad 2: Net-(JP1-B) -> Net-(J5-Pin_1)
- R18 pad 2: Net-(JP1-B) -> Net-(J5-Pin_1)
- R8 pad 2: Net-(JP1-B) -> Net-(J5-Pin_1)
- R9 pad 2: Net-(JP1-B) -> Net-(J5-Pin_1)
- U3 pad A10: unconnected-(U3-P0.29/AIN5-PadA10) -> /COL13
- U3 pad A14: unconnected-(U3-P1.15-PadA14) -> /COL14
- U3 pad A16: unconnected-(U3-P1.13-PadA16) -> /ROW1
- U3 pad A20: unconnected-(U3-P1.10-PadA20) -> /ROW0
- U3 pad A8: unconnected-(U3-P0.31/AIN7-PadA8) -> /COL12
- U3 pad AD10: unconnected-(U3-P0.15-PadAD10) -> /COL5
- U3 pad AD12: unconnected-(U3-P0.17-PadAD12) -> /~{nReset}
- U3 pad AD16: unconnected-(U3-P0.20-PadAD16) -> /COL4
- U3 pad AD18: unconnected-(U3-P0.22-PadAD18) -> /COL3
- U3 pad AD20: unconnected-(U3-P0.24-PadAD20) -> /COL2
- U3 pad AD8: unconnected-(U3-P0.13-PadAD8) -> /COL6
- U3 pad G1: unconnected-(U3-P0.26-PadG1) -> /COL11
- U3 pad J1: unconnected-(U3-P0.04/AIN2-PadJ1) -> /COL10
- U3 pad J24: unconnected-(U3-P0.10/NFC2-PadJ24) -> /ROW2
- U3 pad L1: unconnected-(U3-P0.06-PadL1) -> /COL9
- U3 pad L24: unconnected-(U3-P0.09/NFC1-PadL24) -> /ROW3
- U3 pad N1: unconnected-(U3-P0.08-PadN1) -> /COL8
- U3 pad R1: unconnected-(U3-P1.09/TRACEDATA3-PadR1) -> /COL7
- U3 pad R24: unconnected-(U3-P1.06-PadR24) -> /ROW4
- U3 pad U24: unconnected-(U3-P1.04-PadU24) -> /COL0
- U3 pad W24: unconnected-(U3-P1.02-PadW24) -> /COL1
Routing:
- net /COL13: track 0.00 -> 363.2 mm, vias 0 -> 2
- net /COL12: track 0.00 -> 341.8 mm, vias 0 -> 4
- net /switch_matrix/ROW0: track 0.00 -> 311.1 mm, vias 0 -> 4
- net /COL11: track 0.00 -> 305.6 mm
- net /switch_matrix/ROW3: track 0.00 -> 304.3 mm
- net /COL14: track 0.00 -> 292.5 mm, vias 0 -> 2
- net /switch_matrix/ROW4: track 0.00 -> 289.2 mm
- net /switch_matrix/ROW2: track 0.00 -> 288.0 mm
- net /COL10: track 0.00 -> 281.5 mm
- net /switch_matrix/ROW1: track 0.00 -> 259.6 mm
- net /COL9: track 0.00 -> 241.4 mm
- net /COL6: track 0.00 -> 228.1 mm, vias 0 -> 2
- net /COL8: track 0.00 -> 221.9 mm
- net /COL7: track 0.00 -> 202.4 mm
- net /COL2: track 0.00 -> 179.2 mm, vias 0 -> 4
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- added copper zone on B.Cu, net /USB and Power management/5V
- added copper zone on B.Cu, net /USB and Power management/V_BATT
- added copper zone on B.Cu, net GND
- added copper zone on F.Cu, net GND
- added copper zone on B.Cu, net GNDPWR
- added copper zone on F.Cu, net GNDPWR

Commit message: Completed routing and solved DRC
Parts:
- added G***: LOGO, keyboard:logo-silkscreen, B.Cu at (243.1, 165.6)
- added G***: LOGO, keyboard:keyboard-name-silkscreen, B.Cu at (241.9, 174.7)
- added G***: LOGO, keyboard:creator_logo, B.Cu at (182.0, 177.0)
- added J1: JST-4-pin, keyboard:JST-4-pin, B.Cu at (184.4, 125.6)
- added REF**: OSHW-Logo, keyboard:OSHW-Logo, F.Cu at (220.7, 123.6)
- added SW1: MK-12C02-G025, keyboard:SPDT, B.Cu at (129.4, 140.0)
- added kibuzzard-64C2769B: G***, kibuzzard-64C2769B, F.Cu at (211.2, 125.1)
- MX68: value 1.5u -> 1u; footprint keyboard:SW_Cherry_MX_1.50u_PCB -> keyboard:SW_Cherry_MX_1.00u_PCB
- MX73: footprint keyboard:SW_Cherry_MX_1.00u_PCB -> keyboard:SW_Cherry_MX_1.50u_PCB
- moved MX72 9.54 mm to (328.4, 166.8)
- moved MX71 9.52 mm to (304.6, 166.9)
- moved MX70 9.50 mm to (221.1, 171.9)
- moved MX69 9.50 mm to (142.7, 166.8)
- moved MX73 4.80 mm to (352.2, 166.8)
- moved MX68 4.63 mm to (118.9, 166.8)
- moved JP1 2.52 mm to (83.7, 162.8)
- moved D65 2.30 mm to (341.4, 171.2)
- moved D64 1.90 mm to (317.8, 171.0)
- moved D2 1.85 mm to (131.7, 132.5)
- moved D63 1.13 mm to (294.2, 171.0)
- moved D1 0.96 mm to (129.2, 132.5)
- moved TH1 0.51 mm to (130.1, 124.0)
- moved MX67 0.17 mm to (95.1, 166.8)
- moved Y2 0.16 mm to (109.8, 121.5)
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Connections:
- C1 pad 1: /VBUS -> /USB and Power management/CHG_IN
- J3 pad 10: unconnected-(J3-Pin_10-Pad10) -> /VDD_nRF
- J3 pad 2: /3V3 -> /DB_SWO
- J3 pad 3: /DB_SWDIO -> unconnected-(J3-Pin_3-Pad3)
- J3 pad 4: GND -> unconnected-(J3-Pin_4-Pad4)
- J3 pad 5: /DB_SWO -> GND
- J3 pad 6: unconnected-(J3-Pin_6-Pad6) -> /DB_SWDIO
- JP1 pad 1: /3V3 -> /VDD_nRF
- U1 pad 13: /VBUS -> /USB and Power management/CHG_IN
Routing:
- net /VBUS: track 97.5 -> 200.4 mm, vias 8 -> 9
- net /USB_D+: track 85.3 -> 174.7 mm, vias 5 -> 6
- net /USB_D-: track 83.1 -> 170.9 mm, vias 5 -> 6
- net /VDD_nRF: track 85.6 -> 134.6 mm, vias 7 -> 9
- net /USB and Power management/CHG_IN: track 0.00 -> 41.6 mm, vias 0 -> 2
- net /USB and Power management/5V: track 13.3 -> 28.6 mm, vias 2 -> 4
- net /DB_SWDIO: track 22.4 -> 35.6 mm, vias 0 -> 2
- net /COL2: track 179.2 -> 169.1 mm
- net /3V3: track 9.59 -> 0.00 mm
- net /DB_SWO: track 18.3 -> 27.8 mm, vias 0 -> 3
- net Net-(D61-A): track 27.2 -> 17.7 mm
- net /COL6: track 228.1 -> 218.6 mm
- net Net-(D60-A): track 16.8 -> 7.32 mm
- net Net-(D63-A): track 12.5 -> 6.32 mm
- net /COL11: track 305.6 -> 299.7 mm
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Other:
- board text added: "3V3"
- board text added: "BAT + USB"
- board text added: "CLK"
- board text added: "Designed by Sris"
- board text added: "GND"
- board text added: "IO"
- board text added: "MX70"
- board text added: "ONLY"
- board text added: "Powered by"
- board text added: "RST"
- board text added: "SWO"
- board text added: "USB"
- board text added: "Version 1.0"
- board text added: "X"

Commit message: gerber generated
Parts:
- removed R6, R7: 22E, keyboard:R_0402_1005Metric
- removed REF**: OSHW-Logo, keyboard:OSHW-Logo
- C5, C6, C7, C8: value 100nF -> 8pF
- D10, D11, D12, D13, D14, D15, D16, D17, D18, D19, D20, D21, D22, D23, D24, D25, D26, D27, D28, D29, D3, D30, D31, D32, D33, D34, D35, D36, D37, D38, D39, D4, D40, D41, D42, D43, D44, D45, D46, D47, D48, D49, D5, D50, D51, D52, D53, D54, D55, D56, D57, D58, D59, D6, D60, D61, D62, D63, D64, D65, D7, D8, D9: value 1N4148 -> 1N4148W
- MX73: value 1u -> 1.5u
- U2: value AP2127K-3.0TRG1 -> AP2127K-3.3TRG1
- U3: value NRF52840-QIAA-R -> nRF52840-QIAA-R/nRF52833-QIAA-R
- moved MX31 43.8 mm to (67.5, 96.8)
- moved MX35 43.8 mm to (131.9, 96.8)
- moved MX36 43.8 mm to (151.0, 96.8)
- moved MX37 43.8 mm to (169.9, 96.8)
- moved MX38 43.8 mm to (188.9, 96.8)
- moved MX39 43.8 mm to (208.1, 96.8)
- moved MX40 43.8 mm to (227.1, 96.8)
- moved MX41 43.8 mm to (246.1, 96.8)
- moved MX42 43.8 mm to (265.1, 96.8)
- moved MX43 43.8 mm to (284.1, 96.8)
- moved MX44 43.8 mm to (315.1, 96.8)
- moved MX45 43.8 mm to (72.2, 115.8)
- moved MX48 43.8 mm to (141.3, 115.8)
- moved MX49 43.8 mm to (160.4, 115.8)
- moved MX50 43.8 mm to (179.5, 115.8)
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Connections:
- U3 pad AD4: Net-(U3-D-) -> /USB_D-
- U3 pad AD6: Net-(U3-D+) -> /USB_D+
Routing:
- net /USB_D-: track 170.9 -> 174.6 mm
- net /USB_D+: track 174.7 -> 177.6 mm
- net Net-(U3-D-): track 2.28 -> 0.00 mm
- net Net-(U3-D+): track 2.09 -> 0.00 mm
- net GND: vias 101 -> 102

Commit message: Made changes to add support for salvation keyboard case and discord reviews implemented
Parts:
- removed C15: DNP, keyboard:C_0402_1005Metric
- removed C3, C4: 1uF, keyboard:C_0603_1608Metric
- removed U2: AP2127K-3.3TRG1, keyboard:SOT-23-5
- removed kibuzzard-64C2769B: G***, kibuzzard-64C2769B
- added C17: 100nF, keyboard:C_0402_1005Metric, B.Cu at (20.8, 37.0)
- added H1: MountingHole, keyboard:salvation_mounting_holes, F.Cu at (7.28, -20.6)
- added H2: MountingHole, keyboard:salvation_mounting_holes, F.Cu at (266.0, 34.8)
- added L3: 10uH, keyboard:L_0603_1608Metric, B.Cu at (30.1, 34.0)
- added L4: 15nH, keyboard:L_0402_1005Metric, B.Cu at (30.1, 31.4)
- added L5: 10uH, keyboard:L_0603_1608Metric, B.Cu at (32.6, 42.0)
- added SW2: Reset Switch, keyboard:RST_SW, B.Cu at (34.5, 66.9)
- added kibuzzard-64CB1AC3: G***, kibuzzard-64CB1AC3, B.Cu at (34.6, 70.4)
- moved J1 131.7 mm to (47.0, 17.5)
- moved D17 73.8 mm to (270.5, 12.5)
- moved SW1 73.4 mm to (49.8, 53.9)
- moved MX31 72.6 mm to (19.3, 42.6)
- moved D29 72.5 mm to (224.4, 21.7)
- moved D31 72.5 mm to (267.6, 21.7)
- moved D38 72.5 mm to (130.1, 46.8)
- moved D39 72.5 mm to (149.1, 46.8)
- moved D55 72.5 mm to (216.1, 65.8)
- moved D57 72.5 mm to (268.3, 65.8)
- moved D64 72.5 mm to (239.7, 84.8)
- moved G*** 72.5 mm to (165.0, 79.4)
- moved JP1 72.5 mm to (5.60, 76.6)
- moved MX10 72.5 mm to (183.2, 4.50)
- moved MX14 72.5 mm to (259.7, 4.50)
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Connections:
- C12 pad 2: Net-(U3-DEC4) -> Net-(U3-DEC2)
- J1 pad 1: /VBUS -> /USB and Power management/VBUS
- J4 pad A4: /VBUS -> /USB and Power management/VBUS
- J4 pad B4: /VBUS -> /USB and Power management/VBUS
- R1 pad 1: /USB and Power management/5V -> /VBUS
- R2 pad 1: /USB and Power management/5V -> /VBUS
- SW1 pad 1: /USB and Power management/5V -> /VBUS
- SW1 pad 2: /VBUS -> /USB and Power management/VBUS
- U1 pad 10: /USB and Power management/5V -> /VBUS
- U1 pad 11: /USB and Power management/5V -> /VBUS
- U1 pad 5: /USB and Power management/5V -> /VBUS
- U3 pad AB2: unconnected-(U3-DCCH-PadAB2) -> Net-(U3-DCCH)
- U3 pad AD16: /COL4 -> /COL1
- U3 pad AD18: /COL3 -> /COL4
- U3 pad AD20: /COL2 -> /COL3
- U3 pad B3: unconnected-(U3-DCC-PadB3) -> Net-(U3-DCC)
- U3 pad W24: /COL1 -> /COL2
- U3 pad Y2: /VDD_nRF -> /VBUS
Routing:
- net /VBUS: track 200.4 -> 65.4 mm, vias 9 -> 7
- net /USB and Power management/VBUS: track 0.00 -> 115.9 mm, vias 0 -> 4
- net /USB_D+: track 177.6 -> 91.2 mm, vias 6 -> 4
- net /USB_D-: track 174.6 -> 90.3 mm, vias 6 -> 4
- net /switch_matrix/ROW0: track 311.1 -> 276.6 mm, vias 4 -> 0
- net /COL0: track 139.8 -> 171.8 mm
- net /USB and Power management/5V: track 28.6 -> 0.00 mm, vias 4 -> 0
- net /~{nReset}: track 74.7 -> 101.7 mm, vias 5 -> 8
- net /DB_SWDIO: track 35.6 -> 19.0 mm, vias 2 -> 1
- net /USB and Power management/CHG_IN: track 41.6 -> 28.5 mm
- net /switch_matrix/ROW4: track 286.2 -> 274.5 mm
- net /COL1: track 149.7 -> 138.7 mm, vias 4 -> 2
- net Net-(J5-Pin_1): track 30.8 -> 20.9 mm, vias 3 -> 5
- net /switch_matrix/ROW1: track 259.6 -> 267.4 mm, vias 0 -> 2
- net /ROW4: track 58.5 -> 64.9 mm
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- added copper zone on B.Cu, net /VBUS
- removed copper zone on B.Cu, net /USB and Power management/5V
Other:
- outline, holes or cut-outs redrawn
- board text removed: "Powered by"
